File: connectors.kicad_sch (KiCad schematic)
At the start: 10 parts, among them J1 5V GND, J14 VIA1_IRQB, J15 Conn_01x16_Socket, J2 5V GND, J3 Conn_01x16_Socket, J4 5V GND, J5 Conn_01x08_Socket, J6 VIA0_IRQB, J7 5V GND, J8 Conn_01x08_Socket

Commit message: feat: add proper headers
Parts:
- J1, J2, J4, J7: footprint Connector_PinSocket_2.54mm:PinSocket_1x02_P2.54mm_Vertical -> LCSCLib:HDR-TH_2P-P2.54-V-F-1
- J14, J6: footprint Connector_PinSocket_2.54mm:PinSocket_2x02_P2.54mm_Vertical -> LCSCLib:HDR-TH_4P-P2.54-V-F-R2-C2-S2.54
- J15, J3: footprint Connector_PinSocket_2.54mm:PinSocket_1x16_P2.54mm_Vertical -> LCSCLib:HDR-TH_16P-P2.54-V-F-4
- J5, J8: footprint Connector_PinSocket_2.54mm:PinSocket_1x08_P2.54mm_Vertical -> LCSCLib:HDR-TH_8P-P2.54-V-F
Changed lines of the file:
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@@
 			)
 		)
-		(property "Footprint" "Connector_PinSocket_2.54mm:PinSocket_1x02_P2.54mm_Vertical"
+		(property "Footprint" "LCSCLib:HDR-TH_2P-P2.54-V-F-1"
 			(at 26.67 148.59 0)
 			(effects
@@
 			)
 		)
-		(property "Footprint" "Connector_PinSocket_2.54mm:PinSocket_1x16_P2.54mm_Vertical"
+		(property "Footprint" "LCSCLib:HDR-TH_16P-P2.54-V-F-4"
 			(at 85.09 102.87 0)
 			(effects
@@
 			)
 		)
-		(property "Footprint" "Connector_PinSocket_2.54mm:PinSocket_1x02_P2.54mm_Vertical"
+		(property "Footprint" "LCSCLib:HDR-TH_2P-P2.54-V-F-1"
 			(at 26.67 158.75 0)
 			(effects
@@
 			)
 		)
-		(property "Footprint" "Connector_PinSocket_2.54mm:PinSocket_1x02_P2.54mm_Vertical"
+		(property "Footprint" "LCSCLib:HDR-TH_2P-P2.54-V-F-1"
 			(at 26.67 138.43 0)
 			(effects
@@
 			)
 		)
-		(property "Footprint" "Connector_PinSocket_2.54mm:PinSocket_1x02_P2.54mm_Vertical"
+		(property "Footprint" "LCSCLib:HDR-TH_2P-P2.54-V-F-1"
 			(at 26.67 168.91 0)
 			(effects
@@
 			)
 		)
-		(property "Footprint" "Connector_PinSocket_2.54mm:PinSocket_1x16_P2.54mm_Vertical"
+		(property "Footprint" "LCSCLib:HDR-TH_16P-P2.54-V-F-4"
 			(at 36.83 102.87 0)
 			(effects
@@
 			)
 		)
-		(property "Footprint" "Connector_PinSocket_2.54mm:PinSocket_2x02_P2.54mm_Vertical"
+		(property "Footprint" "LCSCLib:HDR-TH_4P-P2.54-V-F-R2-C2-S2.54"
 			(at 118.11 81.28 0)
 			(effects
@@
 			)
 		)
-		(property "Footprint" "Connector_PinSocket_2.54mm:PinSocket_1x08_P2.54mm_Vertical"
+		(property "Footprint" "LCSCLib:HDR-TH_8P-P2.54-V-F"
 			(at 77.47 19.05 0)
 			(effects
@@
 			)
 		)
-		(property "Footprint" "Connector_PinSocket_2.54mm:PinSocket_2x02_P2.54mm_Vertical"
+		(property "Footprint" "LCSCLib:HDR-TH_4P-P2.54-V-F-R2-C2-S2.54"
 			(at 73.66 81.28 0)
 			(effects
@@
 			)
 		)
-		(property "Footprint" "Connector_PinSocket_2.54mm:PinSocket_1x08_P2.54mm_Vertical"
+		(property "Footprint" "LCSCLib:HDR-TH_8P-P2.54-V-F"
 			(at 77.47 48.26 0)
 			(effects
